File: M-Control-Shield/M-Control-Shield.kicad_pcb (KiCad board)
At the start: 2 copper layers, 71.1 x 66 mm, 4 parts, among them J1 Conn_01x08, J2 Conn_01x06, J3 Conn_01x10, J4 Conn_01x08

Commit message: Annotated and imported to pcb
Parts:
- added C1: C, Capacitor_SMD:C_0603_1608Metric, F.Cu at (210.8, 119.4)
- added C2: C, Capacitor_SMD:C_0603_1608Metric, F.Cu at (231.2, 99.1)
- added C3: C, Capacitor_SMD:C_0603_1608Metric, F.Cu at (214.9, 116.1)
- added C4: C, Capacitor_SMD:C_0603_1608Metric, F.Cu at (214.9, 113.6)
- added C5: C, Capacitor_SMD:C_0603_1608Metric, F.Cu at (210.8, 116.9)
- added C6: C, Capacitor_SMD:C_0603_1608Metric, F.Cu at (223.3, 107.2)
- added C7: C, Capacitor_SMD:C_0603_1608Metric, F.Cu at (226.8, 102.1)
- added D1: SB10150, Diode_THT:D_DO-201AD_P12.70mm_Horizontal, F.Cu at (185.5, 103.7)
- added D2: SB10150, Diode_THT:D_DO-201AD_P12.70mm_Horizontal, F.Cu at (185.5, 96.9)
- added D3: SB10150, Diode_THT:D_DO-201AD_P12.70mm_Horizontal, F.Cu at (202.9, 90.2)
- added D4: SB10150, Diode_THT:D_DO-201AD_P12.70mm_Horizontal, F.Cu at (185.5, 90.2)
- added J5: Conn_02x06_Row_Letter_First, Connector_PinHeader_1.27mm:PinHeader_2x06_P1.27mm_Vertical, F.Cu at (209.5, 107.6)
- added J6: Screw_Terminal_01x02, TerminalBlock_Phoenix:TerminalBlock_Phoenix_PT-1,5-2-5.0-H_1x02_P5.00mm_Horizontal, F.Cu at (216.2, 99.9)
- added J7: Screw_Terminal_01x02, TerminalBlock_Phoenix:TerminalBlock_Phoenix_PT-1,5-2-5.0-H_1x02_P5.00mm_Horizontal, F.Cu at (233.7, 91.8)
- added Q1: AOD413A, Package_TO_SOT_SMD:TO-252-2, F.Cu at (152.4, 104.1)
- added Q2: AOD454A, Package_TO_SOT_SMD:TO-252-2, F.Cu at (189.2, 111.1)
- added Q3: AOD413A, Package_TO_SOT_SMD:TO-252-2, F.Cu at (201.3, 111.1)
- added Q4: AOD454A, Package_TO_SOT_SMD:TO-252-2, F.Cu at (152.4, 94.0)
- added R1: R, Resistor_SMD:R_0805_2012Metric, F.Cu at (226.9, 99.3)
- added R2: R, Resistor_SMD:R_0805_2012Metric, F.Cu at (207.9, 103.1)
- added R3: R, Resistor_SMD:R_0805_2012Metric, F.Cu at (202.2, 116.6)
- added R4: R, Resistor_SMD:R_0805_2012Metric, F.Cu at (206.6, 117.1)
- added R5: R, Resistor_SMD:R_0805_2012Metric, F.Cu at (202.2, 119.5)
- added R6: R, Resistor_SMD:R_0805_2012Metric, F.Cu at (226.9, 96.3)
- added R7: R, Resistor_SMD:R_0805_2012Metric, F.Cu at (206.6, 120.0)
- added U1: SN74LVC1G374, Package_TO_SOT_SMD:SOT-23-6, F.Cu at (203.1, 103.8)
- added U2: MAX17601, Package_SO:SO-8_3.9x4.9mm_P1.27mm, F.Cu at (217.1, 109.1)
- added U3: INA240A4D, Package_SO:SOIC-8_3.9x4.9mm_P1.27mm, F.Cu at (187.3, 118.3)
- added U4: MAX17601, Package_SO:SO-8_3.9x4.9mm_P1.27mm, F.Cu at (195.8, 118.3)
Connections:
- net /GND renamed GND
- J1 pad 4: /+3V3 -> +3.3V
- J2 pad 2: /A1 -> /A0
- J3 pad 6: /D12 -> /COMP1_OUT
- J4 pad 8: /D0 -> unconnected-(J4-Pad8)

Commit message: Placement of FETs, connectors, and current measurement circuit
Parts:
- moved J7 90.8 mm to (142.8, 93.3), turned to 180 degrees
- moved J6 90.8 mm to (137.2, 144.8)
- moved U2 89.6 mm to (128.3, 120.7)
- moved J5 69.2 mm to (141.0, 116.8)
- moved C4 64.5 mm to (153.0, 95.2), turned to -90 degrees
- moved C3 63.6 mm to (156.8, 90.2), turned to 180 degrees
- moved R5 60.0 mm to (147.3, 95.2), turned to 90 degrees
- moved Q2 60.0 mm to (132.1, 129.5)
- moved R4 59.3 mm to (150.5, 97.8), turned to 180 degrees
- moved R3 57.0 mm to (150.5, 92.7), turned to 180 degrees
- moved Q3 50.6 mm to (150.7, 111.5), turned to 180 degrees
- moved U4 40.9 mm to (154.9, 120.7)
- moved U3 38.2 mm to (156.8, 95.2), turned to 90 degrees
- moved C7 34.3 mm to (195.0, 115.1)
- moved C2 34.3 mm to (199.4, 112.2)
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